File: kicad/mixer-controller/mixer-controller.kicad_sch (KiCad schematic)
At the start: 20 parts, among them J1 RS485, J2 CAN, J3 ADC, J4 PWR_IN, J5 CAN, U2 AP1117-50, U3 TJA1050, U4 ESP32-DEVKITC-32U

Commit message: Added encoder breakout and updated other projects
Parts:
- removed C1: 10u, Capacitor_SMD:C_0805_2012Metric, symbol Device:C
- removed U2: AP1117-50, Package_TO_SOT_SMD:SOT-223-3_TabPin2, symbol Regulator_Linear:AP1117-50
- added J6: FAN, Connector_JST:JST_XH_B2B-XH-AM_1x02_P2.50mm_Vertical, symbol Connector:Conn_01x02_Pin
- added J7: 5V, Connector_JST:JST_XH_B2B-XH-A_1x02_P2.50mm_Vertical, symbol Connector:Conn_01x02_Pin
- added Q1: NCEP60T20, Package_TO_SOT_THT:TO-220-3_Vertical, symbol Simulation_SPICE:NMOS
- added R5: 1k, Resistor_SMD:R_0805_2012Metric_Pad1.20x1.40mm_HandSolder, symbol Device:R
- H1, H2, H3, H4: footprint MountingHole:MountingHole_3.2mm_M3 -> MountingHole:MountingHole_3.2mm_M3_Pad_Via
- J4: value PWR_IN -> 12V
Connections:
- net +12V: now also J6.2 (Pin_2)
- net +5V: now also J7.2 (Pin_2)
- net CAN_H: now also J2.2 (Pin_2), J5.2 (Pin_2); no longer J2.1 (Pin_1), J5.1 (Pin_1)
- net CAN_L: now also J2.1 (Pin_1), J5.1 (Pin_1); no longer J2.2 (Pin_2), J5.2 (Pin_2)
- net ESP_CAN_RX: now also U4.28 (IO17); no longer U4.27 (IO16)
- net ESP_CAN_TX: now also U4.27 (IO16); no longer U4.28 (IO17)
- net GND: now also J7.1 (Pin_1), Q1.3 (S)
- net ESP_GPIO_FAN: now reaches U4.10 (IO26)
- net ESP_GPIO_FAN: now also R5.2
- new net: J6.1 (Pin_1), Q1.1 (D)
- new net: Q1.2 (G), R5.1
Other:
- note added: "FAN CONTROL"
- note added: "L-Pass filter implemented on separate board. These components can be left unsoldered."
- moved on the sheet: C2, J4

Commit message: Final updates for manufacturing
Parts:
- J6: footprint Connector_JST:JST_XH_B2B-XH-AM_1x02_P2.50mm_Vertical -> Connector_JST:JST_XH_B2B-XH-A_1x02_P2.50mm_Vertical
Changed lines of the file:
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@@
       (effects (font (size 1.27 1.27)) (justify right))
     )
-    (property "Footprint" "Connector_JST:JST_XH_B2B-XH-AM_1x02_P2.50mm_Vertical" (at 58.42 119.38 0)
+    (property "Footprint" "Connector_JST:JST_XH_B2B-XH-A_1x02_P2.50mm_Vertical" (at 58.42 119.38 0)
       (effects (font (size 1.27 1.27)) hide)
     )
